File: pcbs/power/power_board.kicad_sch (KiCad schematic)
At the start: 37 parts, among them J1 PinSocket_1x04_P2.54, J10 MR30PW-M, J11 MR30PW-M, J12 12V connection, J2 PinSocket_1x04_P2.54, J3 PinSocket_1x04_P2.54, J4 JST_XH_B3B, J5 JST_XH_B3B, J6 XT30PW-F, J7 XT30PW-F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

Commit message: Updated Power-Board PCB design
Parts:
- removed C2, C3, C4: 100nF, PCM_Capacitor_THT_AKL:C_Disc_D5.0mm_W2.5mm_P5.00mm, symbol PCM_Capacitor_AKL:C_Generic
- removed J1, J2, J3: PinSocket_1x04_P2.54, Connector_PinSocket_2.54mm:PinSocket_1x04_P2.54mm_Vertical, symbol Connector_Generic:Conn_01x04
Connections:
- no-connect marks 3 -> 0
Other:
- added sheet VOLTAGE CONVERTER (untitled.kicad_sch)
- note removed: "Connection to DC-DC buck converters"
- moved on the sheet: H1, H2, H3, J8
